File: pcb/microcontroller.sch (KiCad schematic (older format))
At the start: 0 parts

Commit message: AFE mostly complete
Parts:
- added C15, C16, C24, C25: 2.2u, symbol Device:C_Small
- added C17, C18, C19, C20, C21, C23: 0.1u, symbol Device:C_Small
- added C22: 1u, symbol Device:C_Small
- added R13, R14, R15: 10k, symbol Device:R_US
- added R16, R17: 22, symbol Device:R_US
- added R18: 120, symbol Device:R_US
- added U2: STM32F405RGTx, Package_QFP:LQFP-64_10x10mm_P0.5mm, symbol MCU_ST_STM32F4:STM32F405RGTx
- added U3: TCAN330, symbol Interface_CAN_LIN:TCAN330
Connections:
- new net: R15.1, U2.7 (NRST)
- new net: R14.1, U2.60 (BOOT0)
- new net: C25.2, U2.47 (VCAP_2)
- new net: C24.2, U2.31 (VCAP_1)
- new net: R16.2, U2.44 (PA11)
- new net: R17.2, U2.45 (PA12)
- new net +3V3: C15.2, C16.2, C17.2, C18.2, C19.2, C20.2, C21.2, C22.2, C23.2, R15.2, U2.1 (VBAT), U2.13 (VDDA), U2.19 (VDD), U2.32 (VDD), U2.48 (VDD), U2.64 (VDD)
- new net BOOT2: R13.1, U2.28 (PB2)
- new net CAN2_RX: U2.57 (PB5), U3.4 (RXD)
- new net CAN2_TX: U2.34 (PB13), U3.1 (TXD)
- new net CAN_H: R18.1, U3.7 (CANH)
- new net CAN_L: R18.2, U3.6 (CANL)
- new net CS: U2.41 (PA8)
- new net GND: C15.1, C16.1, C17.1, C18.1, C19.1, C20.1, C21.1, C22.1, C23.1, C24.1, C25.1, R13.2, R14.2, U2.12 (VSSA), U2.18 (VSS), U2.63 (VSS)
- new net SPI1_CLK: U2.21 (PA5)
- new net SPI1_MISO: U2.22 (PA6)
- new net SPI1_MOSI: U2.23 (PA7)
- new net UART1_RX: U2.43 (PA10)
- new net UART1_TX: U2.42 (PA9)
- new net UDB_DM: R17.1
- new net USB_DP: R16.1
Other:
- note added: "Bulk Bypass"
- note added: "VDD Pin Bypass"
- note added: "VDDA Bypass"
