File: pcb/bms/bms.sch (KiCad schematic (older format))
At the start: 14 parts, among them J12 Taps 6-8, J13 Taps 0-5, J14 USB_B_Micro, J15 Thermistor 1, J16 Thermistor 2, J17 Deutsch DTP

Commit message: pretty much ready to go
Parts:
- removed H9: MountingHole, MountingHole:MountingHole_3.2mm_M3, symbol Mechanical:MountingHole
- removed J14: USB_B_Micro, Connect:USB_Micro-B_10103594-0001LF, symbol Connector:USB_B_Micro
- removed J16: Thermistor 2, symbol Connector:Conn_01x02_Female
- removed J17: Deutsch DTP, symbol Connector_Generic:Conn_02x02_Top_Bottom
- added C18, C23: 100n, Capacitor_SMD:C_0805_2012Metric, symbol Device:C_Small
- added J10: Signals, Connector_Hirose:Hirose_DF62WZ-9P-2.2DSA, symbol Connector_Generic:Conn_2Rows-09Pins
- added J3: Taps 9-10, Connector_PinHeader_2.54mm:PinHeader_1x02_P2.54mm_Vertical, symbol Connector:Conn_01x02_Male
- added J4: Batt- Out, farasis_p10a_pack:74651195R, symbol Connector_Generic:Conn_01x01
- added J5: Batt+ In, farasis_p10a_pack:74651195R, symbol Connector_Generic:Conn_01x01
- added J6: Batt- In, farasis_p10a_pack:74651195R, symbol Connector_Generic:Conn_01x01
- added J7: Batt+ Out, farasis_p10a_pack:74651195R, symbol Connector_Generic:Conn_01x01
- C30, C31: MPN (none) -> CL21B104KCFSFNE; Manufacturer (none) -> Samsung Electro-Mechanics
- J9: renamed from J15; value Thermistor 1 -> Thermistors; footprint (none) -> Connector_JST:JST_NSH_SM04B-NSHSS-TB_1x04-1MP_P1.00mm_Vertical; symbol Connector:Conn_01x02_Female -> Connector_Generic:Conn_01x04; MPN (none) -> SM04B-NSHSS-TB (LF)(SN); Manufacturer (none) -> JST
- renumbered J13 to J1, J12 to J2
Connections:
- net +BATT: now also J7.1 (Pin_1)
- net -BATT: now also J4.1 (Pin_1)
- net Cell Measurement/TS1: now also J9.3 (Pin_3), C18.1; no longer J9.1 (Pin_1)
- net Cell Measurement/TS3: now also J9.2 (Pin_2), C23.2
- net GND: now also J9.1 (Pin_1), J9.4 (Pin_4), C18.2, C23.1, J10.1 (Pin_1), J10.2 (Pin_2), J6.1 (Pin_1); no longer J9.2 (Pin_2)
- net Microcontroller/USB_DM: now also J10.9 (Pin_9)
- new net +3V3: J10.3 (Pin_3)
- new net BATT+_CONST: J5.1 (Pin_1)
- new net Cell Measurement/C10: J3.1 (Pin_1)
- new net Cell Measurement/C9: J3.2 (Pin_2)
- new net RST_SHUT: J10.5 (Pin_5)
- new net RX: J10.8 (Pin_8)
- new net TX: J10.7 (Pin_7)
- new net USB_DP: J10.6 (Pin_6)
- new net WAKE: J10.4 (Pin_4)
- no-connect marks 1 -> 0
Other:
- note removed: "USART\nUSB\nWAKE\nRST_SHUT\n3v3 external feed\nGround x2"

Commit message: rev1 as manufactured
Parts:
- removed E1: SPARK_GAP, symbol Device:SPARK_GAP
- added D9: 48V, Diode_SMD:D_SMB, symbol Device:D_TVS
- J4, J5, J6, J7: Manufacturer Würth Elektronik -> Wurth Elektronik
Connections:
- net +BATT: now also D9.2 (A2)
- net -BATT: now also D9.1 (A1)
Changed lines of the file:
@@
 F 3 "~" H 650 650 50  0001 C CNN
 F 4 "" H 650 650 50  0001 C CNN "MPN"
+F 5 "" H 650 650 50  0001 C CNN "Manufacturer"
 	1    650  650
 	1    0    0    -1
@@
 F 3 "~" H 1400 650 50  0001 C CNN
 F 4 "" H 1400 650 50  0001 C CNN "MPN"
+F 5 "" H 1400 650 50  0001 C CNN "Manufacturer"
 	1    1400 650
 	1    0    0    -1
@@
 F 3 "~" H 2150 650 50  0001 C CNN
 F 4 "" H 2150 650 50  0001 C CNN "MPN"
+F 5 "" H 2150 650 50  0001 C CNN "Manufacturer"
 	1    2150 650
 	1    0    0    -1
@@
 F 3 "~" H 2900 650 50  0001 C CNN
 F 4 "" H 2900 650 50  0001 C CNN "MPN"
+F 5 "" H 2900 650 50  0001 C CNN "Manufacturer"
 	1    2900 650
 	1    0    0    -1
@@
 F 2 "Connector_PinHeader_2.54mm:PinHeader_1x05_P2.54mm_Vertical" H 6050 3050 50  0001 C CNN
 F 3 "~" H 6050 3050 50  0001 C CNN
-F 4 "~" H 6050 3050 50  0001 C CNN "MPN"
-F 5 "~" H 6050 3050 50  0001 C CNN "Manufacturer"
+F 4 "" H 6050 3050 50  0001 C CNN "MPN"
+F 5 "" H 6050 3050 50  0001 C CNN "Manufacturer"
 	1    6050 3050
 	-1   0    0    -1
@@
 F 2 "Connector_PinHeader_2.54mm:PinHeader_1x04_P2.54mm_Vertical" H 6050 2600 50  0001 C CNN
 F 3 "~" H 6050 2600 50  0001 C CNN
-F 4 "~" H 6050 2600 50  0001 C CNN "MPN"
-F 5 "~" H 6050 2600 50  0001 C CNN "Manufacturer"
+F 4 "" H 6050 2600 50  0001 C CNN "MPN"
+F 5 "" H 6050 2600 50  0001 C CNN "Manufacturer"
 	1    6050 2600
 	-1   0    0    1
@@
 L power:-BATT #PWR04
 U 1 1 60DA2F2B
-P 7500 3250
-F 0 "#PWR04" H 7500 3100 50  0001 C CNN
-F 1 "-BATT" H 7515 3423 50  0000 C CNN
-F 2 "" H 7500 3250 50  0001 C CNN
-F 3 "" H 7500 3250 50  0001 C CNN
-	1    7500 3250
+P 7500 3300
+F 0 "#PWR04" H 7500 3150 50  0001 C CNN
+F 1 "-BATT" H 7515 3473 50  0000 C CNN
+F 2 "" H 7500 3300 50  0001 C CNN
+F 3 "" H 7500 3300 50  0001 C CNN
+	1    7500 3300
 	-1   0    0    1
 $EndComp
@@
 Wire Wire Line
 	8200 2550 8200 2500
-Wire Wire Line
-	8050 3200 8200 3200
-Wire Wire Line
-	8200 3200 8200 2950
 Connection ~ 8200 2950
-Wire Wire Line
-	7650 3200 7500 3200
-Wire Wire Line
-	7500 3200 7500 3250
-Wire Wire Line
-	7500 2950 7500 3200
-Connection ~ 7500 3200
 $Comp
 L Connector_Generic:Conn_01x04 J9
@@
 	7700 1850 7750 1850
 $Comp
-L Device:SPARK_GAP E1
-U 1 1 60E2F095
-P 7850 3200
-F 0 "E1" H 7850 3390 50  0000 C CNN
-F 1 "SPARK_GAP" H 7850 3299 50  0000 C CNN
-F 2 "" H 7850 3130 50  0001 C CNN
-F 3 "~" V 7850 3200 50  0001 C CNN
-F 4 "" H 7850 3200 50  0001 C CNN "MPN"
-	1    7850 3200
-	1    0    0    -1
-$EndComp
-$Comp
 L power:GND #PWR?
 U 1 1 60B24F80
@@
 F 3 "~" H 7950 1650 50  0001 C CNN
 F 4 "74651195R" H 7950 1650 50  0001 C CNN "MPN"
-F 5 "Würth Elektronik" H 7950 1650 50  0001 C CNN "Manufacturer"
+F 5 "Wurth Elektronik" H 7950 1650 50  0001 C CNN "Manufacturer"
 	1    7950 1650
 	1    0    0    -1
@@
 F 3 "~" H 7950 1850 50  0001 C CNN
 F 4 "74651195R" H 7950 1850 50  0001 C CNN "MPN"
-F 5 "Würth Elektronik" H 7950 1850 50  0001 C CNN "Manufacturer"
+F 5 "Wurth Elektronik" H 7950 1850 50  0001 C CNN "Manufacturer"
 	1    7950 1850
 	1    0    0    -1
@@
 F 3 "~" H 8400 2550 50  0001 C CNN
 F 4 "74651195R" H 8400 2550 50  0001 C CNN "MPN"
-F 5 "Würth Elektronik" H 8400 2550 50  0001 C CNN "Manufacturer"
+F 5 "Wurth Elektronik" H 8400 2550 50  0001 C CNN "Manufacturer"
 	1    8400 2550
 	1    0    0    -1
@@
 F 3 "~" H 7300 2550 50  0001 C CNN
 F 4 "74651195R" H 7300 2550 50  0001 C CNN "MPN"
-F 5 "Würth Elektronik" H 7300 2550 50  0001 C CNN "Manufacturer"
+F 5 "Wurth Elektronik" H 7300 2550 50  0001 C CNN "Manufacturer"
 	1    7300 2550
 	-1   0    0    -1
@@
 Wire Wire Line
 	7500 2950 7500 2550
-Connection ~ 7500 2950
 Wire Wire Line
 	6450 4700 6450 4650
@@
 F 2 "Connector_PinHeader_2.54mm:PinHeader_1x02_P2.54mm_Vertical" H 6050 2150 50  0001 C CNN
 F 3 "~" H 6050 2150 50  0001 C CNN
-F 4 "~" H 6050 2150 50  0001 C CNN "MPN"
-F 5 "~" H 6050 2150 50  0001 C CNN "Manufacturer"
+F 4 "" H 6050 2150 50  0001 C CNN "MPN"
+F 5 "" H 6050 2150 50  0001 C CNN "Manufacturer"
 	1    6050 2150
 	-1   0    0    -1
@@
 Text Label 6650 4650 3    50   ~ 0
 WAKE
+$Comp
+L Device:D_TVS D9
+U 1 1 609E1D69
+P 7850 3250
+F 0 "D9" H 7850 3467 50  0000 C CNN
+F 1 "48V" H 7850 3376 50  0000 C CNN
+F 2 "Diode_SMD:D_SMB" H 7850 3250 50  0001 C CNN
+F 3 "~" H 7850 3250 50  0001 C CNN
+F 4 "SMBJ48A" H 7850 3250 50  0001 C CNN "MPN"
+F 5 "Littelfuse" H 7850 3250 50  0001 C CNN "Manufacturer"
+	1    7850 3250
+	1    0    0    -1
+$EndComp
+Wire Wire Line
+	7500 2950 7500 3250
+Connection ~ 7500 2950
+Wire Wire Line
+	7500 3250 7700 3250
+Connection ~ 7500 3250
+Wire Wire Line
+	7500 3250 7500 3300
+Wire Wire Line
+	8200 2950 8200 3250
+Wire Wire Line
+	8000 3250 8200 3250
 $EndSCHEMATC
