File: pcb/bms/cell_measurement.sch (KiCad schematic (older format))
At the start: 62 parts, among them Q1 FCX495TA, Q2 CSD19506KTT, Q3 CSD19506KTT, Q4 ZXMP10A13FTA, Q5 ZXMP10A13FTA, SW2 SW_Push, U1 BQ76942PFBR

Commit message: split boards to two separate projects
Parts:
- added R12: 20, Resistor_SMD:R_0805_2012Metric, symbol Device:R_US
- C13: value 0.47u -> 470n
- C17: renamed from C?; value 0.1u -> 100n
- C2, C32, C33: value 0.1u -> 100n
- D1, D5: value D -> 100V; footprint (none) -> Diodes_SMD:D_SOD-123; symbol Device:D -> Device:D_Schottky; MPN (none) -> BAT46W-7-F; Manufacturer (none) -> Diodes Inc
- D2, D4: footprint (none) -> Diodes_SMD:D_SOD-123; MPN (none) -> MMSZ5246B-7-F; Manufacturer (none) -> Diodes Inc
- D3: footprint (none) -> Diodes_SMD:D_SOD-123; symbol Device:D_Zener -> Device:D_Schottky; MPN (none) -> BAT46W-7-F; Manufacturer (none) -> Diodes Inc
- Q1: footprint (none) -> TO_SOT_Packages_SMD:SOT-89-3; MPN (none) -> FCX495TA; Manufacturer (none) -> Diodes Inc
- SW2: value SW_Push -> Wake; footprint (none) -> Buttons_Switches_SMD:SW_SPST_PTS645; MPN (none) -> PTS645SK50SMTR92 LFS; Manufacturer (none) -> C&K
- U1: MPN (none) -> https://www.ti.com/store/ti/en/p/product/?p=BQ7694201PFBR; Manufacturer (none) -> TI
- renumbered R12 to R36
Other:
- moved on the sheet: C13

Commit message: pretty much ready to go
Parts:
- added C16: 100n, Capacitor_SMD:C_0805_2012Metric, symbol Device:C_Small
- added C24, C25: 220n, Capacitor_SMD:C_0805_2012Metric, symbol Device:C_Small
- added D8: 5.5V, Package_TO_SOT_SMD:SOT-23, symbol Device:D_TVS_x2_AAC
- added JP7, JP9: Jumper_NO_Small, Jumper:SolderJumper-2_P1.3mm_Open_RoundedPad1.0x1.5mm, symbol Device:Jumper_NO_Small
- added R40, R41: 20, Resistor_SMD:R_0805_2012Metric, symbol Device:R_US
- added SW3: RST, Button_Switch_SMD:SW_SPST_PTS645, symbol Switch:SW_Push
- C1, C12: MPN (none) -> C0805C101J1GACTU; Manufacturer (none) -> Kemet
- C10, C14, C3, C4, C5, C6, C7, C8, C9: MPN (none) -> C0805C224K1RECAUTO; Manufacturer (none) -> Kemet
- C11, C28, C29: MPN (none) -> CL21B105KBFNNNG; Manufacturer (none) -> Samsung Electro-Mechanics
- C13: MPN (none) -> CL21B473KCCWPNC; Manufacturer (none) -> Samsung Electro-Mechanics
- C17, C2, C32, C33: MPN (none) -> CL21B104KCFSFNE; Manufacturer (none) -> Samsung Electro-Mechanics
- C26: MPN (none) -> CL21B223KBANFNC; Manufacturer (none) -> Samsung Electro-Mechanics
- C35: MPN (none) -> CL21B225KPFNNNE; Manufacturer (none) -> Samsung Electro-Mechanics
- Q2, Q3: MPN (none) -> CSD19506KTT; Manufacturer (none) -> TI
- Q4, Q5: MPN (none) -> ZXMP10A13FTA; Manufacturer (none) -> Diodes Inc
- R1, R3, R36: MPN (none) -> CR0805-FX-1000ELF; Manufacturer (none) -> Bourns Inc
- R10, R11, R12, R4, R5, R6, R7, R8, R9: MPN (none) -> RMCF0805FT20R0; Manufacturer (none) -> Stackpole Electronics
- R19, R22, R23, R24, R26, R27: MPN (none) -> RMCF0805FT10K0; Manufacturer (none) -> Stackpole Electronics
- R2: value 2m -> 1m; footprint Resistor_SMD:R_1210_3225Metric -> Resistor_SMD:R_2512_6332Metric; MPN (none) -> CSR2512C0R001F; Manufacturer (none) -> Riedon
- R20, R21: MPN (none) -> RMCF0805FT150R; Manufacturer (none) -> Stackpole Electronics
- R25, R31, R33: MPN (none) -> RMCF0805FT5K10; Manufacturer (none) -> Stackpole Electronics
- R28: MPN (none) -> CR0805-FX-1001ELF; Manufacturer (none) -> Bourns Inc
- R29, R35: MPN (none) -> RMCF0805FT3K90; Manufacturer (none) -> Stackpole Electronics
- R30, R34: MPN (none) -> RMCF0805FT1M00; Manufacturer (none) -> Stackpole Electronics
- R32: MPN (none) -> RMCF0805FT10M0; Manufacturer (none) -> Stackpole Electronics
- SW2: footprint Buttons_Switches_SMD:SW_SPST_PTS645 -> Button_Switch_SMD:SW_SPST_PTS645
- U1: MPN https://www.ti.com/store/ti/en/p/product/?p=BQ7694201PFBR -> BQ7694201PFBR
Connections:
- net +3V3: now also C16.1, SW3.1
- net GND: now also D8.3 (common)
- net RST_SHUT: now also C16.2, D8.2 (A2), SW3.2
- net at C5.2, C7.1, R8.2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: now also JP7.2; no longer U1.2 (VC9), U1.4 (VC8)
- net WAKE: now reaches C17.1, SW2.2, U1.22 (TS2/WAKE)
- net WAKE: now also D8.1 (A1)
- net at C5.1, R6.2: now also U1.4 (VC8), C25.2, JP7.1, JP9.1; no longer U1.48 (VC10)
- new net: C24.2, C25.1, JP9.2, R41.2, U1.2 (VC9)
- new net: C24.1, R40.2, U1.48 (VC10)
- new net C10: R40.1
- new net C9: R41.1
Other:
- note added: "REG1 Bypass"
- moved on the sheet: C28
