File: pcb/cell_interconnect/8S_interconnect.sch (KiCad schematic (older format))
At the start: 22 parts, among them J1 C0, J2 C1, J3 C2, J4 C3, J5 C4, J6 C5, J7 C6, J8 C7, J9 C8

Commit message: rev1 as manufactured
Parts:
- F8: MPN (none) -> C2Q 300; Manufacturer (none) -> Bel Fuse Inc
- J1: footprint farasis_p10a_pack:cell_tap_wire_land -> farasis_p10a_pack:farasis_p10a_end_tab_offset_right
- J9: footprint farasis_p10a_pack:cell_tap_wire_land -> farasis_p10a_pack:farasis_p10a_end_tab_offset_left
Changed lines of the file:
@@
 F 0 "J1" H 4518 4875 50  0000 C CNN
 F 1 "C0" H 4518 4966 50  0000 C CNN
-F 2 "farasis_p10a_pack:cell_tap_wire_land" H 4600 5100 50  0001 C CNN
+F 2 "farasis_p10a_pack:farasis_p10a_end_tab_offset_right" H 4600 5100 50  0001 C CNN
 F 3 "~" H 4600 5100 50  0001 C CNN
 F 4 "~" H 4600 5100 50  0001 C CNN "MPN"
@@
 F 2 "Resistor_SMD:R_0603_1608Metric" V 5230 2650 50  0001 C CNN
 F 3 "~" H 5300 2650 50  0001 C CNN
-F 4 "~" H 5300 2650 50  0001 C CNN "MPN"
+F 4 "C2Q 300" H 5300 2650 50  0001 C CNN "MPN"
+F 5 "Bel Fuse Inc" V 5300 2650 50  0001 C CNN "Manufacturer"
 	1    5300 2650
 	0    1    1    0
@@
 F 0 "J9" H 4518 2075 50  0000 C CNN
 F 1 "C8" H 4518 2166 50  0000 C CNN
-F 2 "farasis_p10a_pack:cell_tap_wire_land" H 4600 2300 50  0001 C CNN
+F 2 "farasis_p10a_pack:farasis_p10a_end_tab_offset_left" H 4600 2300 50  0001 C CNN
 F 3 "~" H 4600 2300 50  0001 C CNN
 F 4 "~" H 4600 2300 50  0001 C CNN "MPN"
