File: pcb/cell_interconnect/cell_interconnect.kicad_pcb (KiCad board)
At the start: 2 copper layers, 80 x 60 mm, 24 parts, among them J1 C0, J10 Taps 6-8, J11 Taps 0-5, J2 C1, J3 C2, J4 C3, J5 C4, J6 C5, J7 C6, J8 C7, J9 C8

Commit message: rev1 as manufactured
Parts:
- J1: footprint farasis_p10a_pack:cell_tap_wire_land -> farasis_p10a_pack:farasis_p10a_end_tab_offset_right
- J9: footprint farasis_p10a_pack:cell_tap_wire_land -> farasis_p10a_pack:farasis_p10a_end_tab_offset_left
- moved F9 11.3 mm to (150.5, 94.0)
- moved F1 10.9 mm to (111.1, 94.0)
- moved J9 1.54 mm to (161.0, 80.9)
- moved J1 1.51 mm to (101.0, 80.9), turned to 270 degrees
- moved F2 0.41 mm to (106.0, 95.5)
- moved F8 0.41 mm to (156.0, 95.5)
Routing:
- net Net-(F1-Pad1): track 9.28 -> 22.7 mm
- net Net-(F9-Pad2): track 9.28 -> 22.6 mm
- net /8S/C8: track 26.8 -> 14.4 mm
- net /8S/C0: track 24.9 -> 13.3 mm
- net Net-(F8-Pad2): track 14.7 -> 16.2 mm
- net /8S/C1: track 24.0 -> 25.2 mm
- net /8S/C7: track 28.1 -> 27.4 mm
